Commit message: initial test shows the jacobian is analytical

File: acrobot/model/gen/models/Acrobot.urdf (robot description, URDF)
Before this commit: robot Acrobot, 3 links, 2 joints
Joints:
- joint jB: origin xyz=-1.00000 0.00000 0.00000 rpy=0.0 0.0 0.0 -> xyz=1.00000 0.00000 0.00000 rpy=0.0 0.0 0.0; type prismatic -> revolute
